Commit message: Optimize URDF for better simulation performance

File: src/terrain_rover_sim/urdf/macros.xacro (robot description, xacro)
@@ -1,14 +1,7 @@
 <?xml version="1.0" encoding="utf-8"?>
 <robot xmlns:xacro="http://www.ros.org/wiki/xacro">
-  <xacro:macro name="leo"
-               params="default_antenna:=true
-                       rockers_fixed:=true
-                       footprint_link:=true
-                       link_prefix:=''
-                       joint_prefix:=''
-                       imu_translation:='0.0628 -0.0314 -0.0393'
-                       mecanum_wheels:=false">
+  <xacro:macro name="rover_base" params="">
     <xacro:macro name="rocker_link" params="name">
-      <link name="${link_prefix}rocker_${name}_link">
+      <link name="rocker_${name}_link">
         <inertial>
           <mass value="1.387336"/>
@@ -21,10 +14,10 @@
         <visual>
           <geometry>
-            <mesh filename="package://leo_description/models/Rocker.dae"/>
+            <mesh filename="package://terrain_rover_sim/models/leo_models/Rocker.dae"/>
           </geometry>
         </visual>
         <collision>
           <geometry>
-            <mesh filename="package://leo_description/models/Rocker_outline.stl"/>
+            <mesh filename="package://terrain_rover_sim/models/leo_models/Rocker_outline.stl"/>
           </geometry>
         </collision>
@@ -32,5 +25,5 @@
     </xacro:macro>
     <xacro:macro name="wheel_link" params="name model">
-      <link name="${link_prefix}wheel_${name}_link">
+      <link name="wheel_${name}_link">
         <inertial>
           <mass value="0.283642"/>
@@ -43,5 +36,5 @@
         <visual>
           <geometry>
-            <mesh filename="package://leo_description/models/Wheel${model}.dae"/>
+            <mesh filename="package://terrain_rover_sim/models/leo_models/Wheel${model}.dae"/>
           </geometry>
         </visual>
@@ -58,44 +51,9 @@
           </geometry>
         </collision>
-        <collision>
-          <geometry>
-            <mesh filename="package://leo_description/models/Wheel_outline.stl"/>
-          </geometry>
-        </collision>
-      </link>
-    </xacro:macro>
-    <xacro:macro name="mecanum_wheel_link" params="name model">
-      <link name="${link_prefix}wheel_${name}_link">
-        <inertial>
-          <mass value="0.672214"/>
-          <origin xyz="0 -0.036852 0"/>
-          <inertia
-            ixx="0.0009778"  ixy="-8.10228e-7" ixz="3.2e-11"
-            iyy="0.001321" iyz="5.7e-11"
-            izz="0.0009773"/>
-        </inertial>
-        <visual>
-          <geometry>
-            <mesh filename="package://leo_description/models/WheelMecanum${model}.dae"/>
-          </geometry>
-        </visual>
-        <collision>
-          <origin xyz="0 -0.0317 0" rpy="${pi/2} 0 0"/>
-          <geometry>
-            <cylinder radius="0.0635" length="0.0515"/>
-          </geometry>
-        </collision>
-        <collision>
-          <geometry>
-            <mesh filename="package://leo_description/models/Mecanum_wheel_outline.stl"/>
-          </geometry>
-        </collision>
       </link>
     </xacro:macro>
     <!-- LINKS -->
-    <xacro:if value="${footprint_link}">
-      <link name="${link_prefix}base_footprint"/>
-    </xacro:if>
-    <link name="${link_prefix}base_link">
+    <link name="base_footprint"/>
+    <link name="base_link">
       <inertial>
         <mass value="1.584994"/>
@@ -108,10 +66,10 @@
       <visual>
         <geometry>
-          <mesh filename="package://leo_description/models/Chassis.dae"/>
+          <mesh filename="package://terrain_rover_sim/models/leo_models/Chassis.dae"/>
         </geometry>
       </visual>
       <collision>
         <geometry>
-          <mesh filename="package://leo_description/models/Chassis_outline.stl"/>
+          <mesh filename="package://terrain_rover_sim/models/leo_models/Chassis_outline.stl"/>
         </geometry>
       </collision>
@@ -119,42 +77,9 @@
     <xacro:rocker_link name="L"/>
     <xacro:rocker_link name="R"/>
-    <xacro:if value="${mecanum_wheels}">
-      <xacro:mecanum_wheel_link name="FL" model="B"/>
-      <xacro:mecanum_wheel_link name="RL" model="A"/>
-      <xacro:mecanum_wheel_link name="FR" model="A"/>
-      <xacro:mecanum_wheel_link name="RR" model="B"/>
-    </xacro:if>
-    <xacro:unless value="${mecanum_wheels}">
-      <xacro:wheel_link name="FL" model="A"/>
-      <xacro:wheel_link name="RL" model="A"/>
-      <xacro:wheel_link name="FR" model="B"/>
-      <xacro:wheel_link name="RR" model="B"/>
-    </xacro:unless>
-    <xacro:if value="${default_antenna}">
-      <link name="${link_prefix}antenna_link">
-        <inertial>
-          <mass value="0.001237"/>
-          <origin xyz="0 0 0.028828"/>
-          <inertia
-            ixx="2.5529e-7" ixy="0.0" ixz="0.0"
-            iyy="2.5529e-7" iyz="0.0"
-            izz="1.354e-8"/>
-        </inertial>
-        <visual>
-          <geometry>
-            <mesh filename="package://leo_description/models/Antenna.dae"/>
-          </geometry>
-        </visual>
-        <collision>
-          <origin xyz="0 0 0.028"/>
-          <geometry>
-            <cylinder radius="0.0055" length="0.056"/>
-          </geometry>
-        </collision>
-      </link>
-    </xacro:if>
-    <link name="${link_prefix}camera_frame"/>
-    <link name="${link_prefix}camera_optical_frame"/>
-    <link name="${link_prefix}depth_camera_frame">
+    <xacro:wheel_link name="FL" model="A"/>
+    <xacro:wheel_link name="RL" model="A"/>
+    <xacro:wheel_link name="FR" model="B"/>
+    <xacro:wheel_link name="RR" model="B"/>
+    <link name="depth_camera_frame">
       <inertial>
         <mass value="0.05"/>
@@ -190,8 +115,7 @@
       </collision>
     </link>
-    <link name="${link_prefix}depth_camera_optical_frame"/>
-    <link name="${link_prefix}imu_frame"/>
-    <!-- LIDAR LINK -->
-    <link name="${link_prefix}lidar_link">
+    <link name="depth_camera_optical_frame"/>
+    <link name="imu_frame"/>
+    <link name="lidar_link">
 			<inertial>
 				<mass value="0.1"/>
@@ -219,29 +143,21 @@
 		</link>
     <!-- JOINTS -->
-    <xacro:if value="${footprint_link}">
-      <joint name="${joint_prefix}base_joint" type="fixed">
-        <origin xyz="0 0 0.19783" rpy="0 0 0"/>
-        <parent link="${link_prefix}base_footprint"/>
-        <child link="${link_prefix}base_link"/>
-      </joint>
-    </xacro:if>
-    <xacro:if value="${rockers_fixed}">
-      <xacro:property name="rockers_joint_type" value="fixed"/>
-    </xacro:if>
-    <xacro:unless value="${rockers_fixed}">
-      <xacro:property name="rockers_joint_type" value="revolute"/>
-    </xacro:unless>
-    <joint name="${joint_prefix}rocker_L_joint" type="${rockers_joint_type}">
+    <joint name="base_joint" type="fixed">
+      <origin xyz="0 0 0.19783" rpy="0 0 0"/>
+      <parent link="base_footprint"/>
+      <child link="base_link"/>
+    </joint>
+    <joint name="rocker_L_joint" type="revolute">
       <origin xyz="0.00263 0.14167 -0.04731" rpy="0 0 ${pi}"/>
-      <parent link="${link_prefix}base_link"/>
-      <child link="${link_prefix}rocker_L_link"/>
+      <parent link="base_link"/>
+      <child link="rocker_L_link"/>
       <axis xyz="0 1 0"/>
       <limit effort="100.0" lower="-0.24" upper="0.24" velocity="100.0"/>
       <dynamics friction="1.0" damping="0.1"/>
     </joint>
-    <joint name="${joint_prefix}rocker_R_joint" type="${rockers_joint_type}">
+    <joint name="rocker_R_joint" type="revolute">
       <origin xyz="0.00263 -0.14167 -0.04731" rpy="0 0 0"/>
-      <parent link="${link_prefix}base_link"/>
-      <child link="${link_prefix}rocker_R_link"/>
+      <parent link="base_link"/>
+      <child link="rocker_R_link"/>
       <axis xyz="0 1 0"/>
       <limit effort="100.0" lower="-0.24" upper="0.24" velocity="100.0"/>
@@ -249,104 +165,61 @@
       <mimic joint="rocker_L_joint"/>
     </joint>
-    <joint name="${joint_prefix}wheel_FL_joint" type="continuous">
-      <xacro:if value="${mecanum_wheels}">
-        <origin xyz="-0.15256 -0.00884 -0.08802" rpy="0 0 0"/>
-      </xacro:if>
-      <xacro:unless value="${mecanum_wheels}">
-        <origin xyz="-0.15256 -0.08214 -0.08802" rpy="0 0 0"/>
-      </xacro:unless>
-      <parent link="${link_prefix}rocker_L_link"/>
-      <child link="${link_prefix}wheel_FL_link"/>
+    <joint name="wheel_FL_joint" type="continuous">
+      <origin xyz="-0.15256 -0.08214 -0.08802" rpy="0 0 0"/>
+      <parent link="rocker_L_link"/>
+      <child link="wheel_FL_link"/>
       <axis xyz="0 -1 0"/>
-      <limit effort="2.0" velocity="6.0"/>
+      <limit effort="2.0" velocity="12.0"/>
       <dynamics friction="0.3125" damping="0.1"/>
     </joint>
-    <joint name="${joint_prefix}wheel_RL_joint" type="continuous">
-      <xacro:if value="${mecanum_wheels}">
-        <origin xyz="0.15256 -0.00884 -0.08802" rpy="0 0 0"/>
-      </xacro:if>
-      <xacro:unless value="${mecanum_wheels}">
-        <origin xyz="0.15256 -0.08214 -0.08802" rpy="0 0 0"/>
-      </xacro:unless>
-      <parent link="${link_prefix}rocker_L_link"/>
-      <child link="${link_prefix}wheel_RL_link"/>
+    <joint name="wheel_RL_joint" type="continuous">
+      <origin xyz="0.15256 -0.08214 -0.08802" rpy="0 0 0"/>
+      <parent link="rocker_L_link"/>
+      <child link="wheel_RL_link"/>
       <axis xyz="0 -1 0"/>
-      <limit effort="2.0" velocity="6.0"/>
+      <limit effort="2.0" velocity="12.0"/>
       <dynamics friction="0.3125" damping="0.1"/>
     </joint>
-    <joint name="${joint_prefix}wheel_FR_joint" type="continuous">
-      <xacro:if value="${mecanum_wheels}">
-        <origin xyz="0.15256 -0.00884 -0.08802" rpy="0 0 0"/>
-      </xacro:if>
-      <xacro:unless value="${mecanum_wheels}">
-        <origin xyz="0.15256 -0.08214 -0.08802" rpy="0 0 0"/>
-      </xacro:unless>
-      <parent link="${link_prefix}rocker_R_link"/>
-      <child link="${link_prefix}wheel_FR_link"/>
+    <joint name="wheel_FR_joint" type="continuous">
+      <origin xyz="0.15256 -0.08214 -0.08802" rpy="0 0 0"/>
+      <parent link="rocker_R_link"/>
+      <child link="wheel_FR_link"/>
       <axis xyz="0 1 0"/>
-      <limit effort="2.0" velocity="6.0"/>
+      <limit effort="2.0" velocity="12.0"/>
       <dynamics friction="0.3125" damping="0.1"/>
     </joint>
-    <joint name="${joint_prefix}wheel_RR_joint" type="continuous">
-      <xacro:if value="${mecanum_wheels}">
-        <origin xyz="-0.15256 -0.00884 -0.08802" rpy="0 0 0"/>
-      </xacro:if>
-      <xacro:unless value="${mecanum_wheels}">
-        <origin xyz="-0.15256 -0.08214 -0.08802" rpy="0 0 0"/>
-      </xacro:unless>
-      <parent link="${link_prefix}rocker_R_link"/>
-      <child link="${link_prefix}wheel_RR_link"/>
+    <joint name="wheel_RR_joint" type="continuous">
+      <origin xyz="-0.15256 -0.08214 -0.08802" rpy="0 0 0"/>
+      <parent link="rocker_R_link"/>
+      <child link="wheel_RR_link"/>
       <axis xyz="0 1 0"/>
-      <limit effort="2.0" velocity="6.0"/>
+      <limit effort="2.0" velocity="12.0"/>
       <dynamics friction="0.3125" damping="0.1"/>
     </joint>
-    <xacro:if value="${default_antenna}">
-      <joint name="${joint_prefix}antenna_joint" type="fixed">
-        <origin xyz="-0.0052 0.056 -0.0065" rpy="0 0 0"/>
-        <parent link="${link_prefix}base_link"/>
-        <child link="${link_prefix}antenna_link"/>
-      </joint>
-    </xacro:if>
-    <joint name="${joint_prefix}camera_joint" type="fixed">
-      <origin xyz="0.0971 0 -0.0427" rpy="0 0.2094 0"/>
-      <parent link="${link_prefix}base_link"/>
-      <child link="${link_prefix}camera_frame"/>
-    </joint>
-    <joint name="${joint_prefix}camera_optical_joint" type="fixed">
+    <joint name="depth_camera_joint" type="fixed">
+      <origin xyz="0.15 0 0.26" rpy="0 0.45 0"/>
+      <parent link="base_link"/>
+      <child link="depth_camera_frame"/>
+    </joint>
+    <joint name="depth_camera_optical_joint" type="fixed">
       <origin xyz="0 0 0" rpy="-${pi/2} 0.0 -${pi/2}"/>
-      <parent link="${link_prefix}camera_frame"/>
-      <child link="${link_prefix}camera_optical_frame"/>
-    </joint>
-    <joint name="${joint_prefix}depth_camera_joint" type="fixed">
-      <origin xyz="0.15 0 0.26" rpy="0 0.45 0"/>
-      <parent link="${link_prefix}base_link"/>
-      <child link="${link_prefix}depth_camera_frame"/>
-    </joint>
-    <joint name="${joint_prefix}depth_camera_optical_joint" type="fixed">
-      <origin xyz="0 0 0" rpy="-${pi/2} 0.0 -${pi/2}"/>
-      <parent link="${link_prefix}depth_camera_frame"/>
-      <child link="${link_prefix}depth_camera_optical_frame"/>
-    </joint>
-    <joint name="${joint_prefix}imu_joint" type="fixed">
-      <origin xyz="${imu_translation}" rpy="0 0 0"/>
-      <parent link="${link_prefix}base_link"/>
-      <child link="${link_prefix}imu_frame"/>
-    </joint>
-    <!-- LIDAR JOINT -->
-    <joint name="${joint_prefix}lidar_joint" type="fixed">
+      <parent link="depth_camera_frame"/>
+      <child link="depth_camera_optical_frame"/>
+    </joint>
+    <joint name="imu_joint" type="fixed">
+      <origin xyz="0.0628 -0.0314 -0.0393" rpy="0 0 0"/>
+      <parent link="base_link"/>
+      <child link="imu_frame"/>
+    </joint>
+    <joint name="lidar_joint" type="fixed">
 			<origin xyz="0.08 0 0.2" rpy="0 0 0"/>
-			<parent link="${link_prefix}base_link"/>
-			<child link="${link_prefix}lidar_link"/>
+			<parent link="base_link"/>
+			<child link="lidar_link"/>
 		</joint>
   </xacro:macro>
-  <!-- LEO GAZEBO -->
-  <xacro:macro name="leo_gazebo"
-               params="robot_ns:='''">
-    <xacro:property name="link_prefix" value=""/>
-    <xacro:if value="${robot_ns != '' and robot_ns != '/'}">
-      <xacro:property name="link_prefix" value="${robot_ns}/"/>
-    </xacro:if>
+  <!-- GAZEBO -->
+  <xacro:macro name="rover_gazebo" params="">
     <!-- base ODE properties -->
-    <gazebo reference="${link_prefix}base_footprint">
+    <gazebo reference="base_footprint">
       <collision>
         <surface>
@@ -365,5 +238,5 @@
       </collision>
     </gazebo>
-    <gazebo reference="${link_prefix}base_link">
+    <gazebo reference="base_link">
       <collision>
         <surface>
@@ -383,5 +256,5 @@
     </gazebo>
     <!-- rocker ODE properties -->
-    <gazebo reference="${link_prefix}rocker_L_link">
+    <gazebo reference="rocker_L_link">
       <collision>
         <surface>
@@ -400,5 +273,5 @@
       </collision>
     </gazebo>
-    <gazebo reference="${link_prefix}rocker_R_link">
+    <gazebo reference="rocker_R_link">
       <collision>
         <surface>
@@ -417,6 +290,6 @@
       </collision>
     </gazebo>
-    <!-- wheel ODE properties -->
-    <gazebo reference="${link_prefix}wheel_FL_link">
+    <!-- wheel properties -->
+    <gazebo reference="wheel_FL_link">
       <collision>
         <surface>
@@ -425,7 +298,4 @@
               <mu>3.0</mu>
               <mu2>3.0</mu2>
-              <slip1>0.005</slip1>
-              <slip2>0</slip2>
-              <fdir1>0 0 1</fdir1>
             </ode>
             <bullet>
@@ -438,5 +308,5 @@
       </collision>
     </gazebo>
-    <gazebo reference="${link_prefix}wheel_FR_link">
+    <gazebo reference="wheel_FR_link">
       <collision>
         <surface>
@@ -445,7 +315,4 @@
               <mu>3.0</mu>
               <mu2>3.0</mu2>
-              <slip1>0.005</slip1>
-              <slip2>0</slip2>
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
File: src/terrain_rover_sim/urdf/rover_sim.urdf.xacro (robot description, xacro)
@@ -2,8 +2,5 @@
 <robot xmlns:xacro="http://ros.org/wiki/xacro"
        name="terrain_rover">
-  <xacro:arg name="fixed" default="false"/>
   <xacro:include filename="$(find terrain_rover_sim)/urdf/macros.xacro"/>
-  <xacro:leo_sim fixed="$(arg fixed)"
-                 robot_ns=""
-                 mecanum_wheels="false"/>
+  <xacro:rover_sim/>
 </robot>
